Commit message: Fix path

File: objects/beer_bottle/beer_bottle.urdf (robot description, URDF)
Before this commit: robot beer_bottle, 3 links, 2 joints
Links:
- link beer_bottle_body: geometry collision mesh filename=file://beer_bottle/meshes/stl/BeerBottleBody_001.stl scale=1.0 1.0 1.0; collision mesh filename=file://beer_bottle/meshes/stl/BeerBottleBody_002.stl scale=1.0 1.0 1.0
- link beer_bottle_cap: geometry collision mesh filename=file://beer_bottle/meshes/stl/BeerBottleCap_001.stl scale=1.0 1.0 1.0; collision mesh filename=file://beer_bottle/meshes/stl/BeerBottleCap_002.stl scale=1.0 1.0 1.0

File: objects/bread_1/bread_1.urdf (robot description, URDF)
Before this commit: robot bread_1, 2 links, 1 joints
Links:
- link bread1: geometry collision mesh filename=file://bread_1/meshes/stl/Bread1_001.stl scale=1.0 1.0 1.0; collision mesh filename=file://bread_1/meshes/stl/Bread1_002.stl scale=1.0 1.0 1.0

File: objects/long_saussage/long_saussage.urdf (robot description, URDF)
Before this commit: robot long_saussage, 1 links, 0 joints
Links:
- link long_saussage: geometry collision mesh filename=file://long_saussage/meshes/stl/LongSaussage_001.stl scale=1.0 1.0 1.0; collision mesh filename=file://long_saussage/meshes/stl/LongSaussage_002.stl scale=1.0 1.0 1.0
