Commit message: Fix bread_1

File: objects/bread_1/bread_1.urdf (robot description, URDF)
Before this commit: robot bread_1, 2 links, 1 joints
Links:
- removed link bread1
- link bread_1: mass None -> 0.8408675193786621; geometry collision mesh filename=file://bread_1/meshes/stl/Bread1_001.stl scale=1.0 1.0 1.0; collision mesh filename=file://bread_1/meshes/stl/Bread1_002.stl scale=1.0 1.0 1.0
Joints:
- removed joint bread1_joint
