Commit message: Fix bread_2

File: objects/bread_2/bread_2.urdf (robot description, URDF)
Before this commit: robot bread_2, 2 links, 1 joints
Links:
- removed link bread2
- link bread_2: mass None -> 0.5353232622146606; geometry collision mesh filename=file://bread_2/meshes/stl/Bread2_001.stl scale=1.0 1.0 1.0; collision mesh filename=file://bread_2/meshes/stl/Bread2_002.stl scale=1.0 1.0 1.0
Joints:
- removed joint bread2_joint
