Commit message: Fix tiago_dual

File: robots/agents/pal_robotics/tiago_dual/tiago_dual.urdf (robot description, URDF)
Before this commit: robot tiago_dual, 70 links, 69 joints
Links:
- link base_link: mass 3.5307810306549072 -> 4.583009719848633; geometry collision mesh filename=file://tiago_dual/meshes/stl/base_collision.stl scale=1.0 1.0 1.0; visual mesh filename=file://tiago_dual/meshes/obj/base.obj scale=1.0 1.0 1.0
- link gripper_left_left_finger_link: mass 8000.0458984375 -> 0.10103759169578552
- link gripper_left_right_finger_link: mass 8000.0458984375 -> 0.10103759169578552
- link gripper_right_left_finger_link: mass 8000.0458984375 -> 0.10103759169578552
- link gripper_right_right_finger_link: mass 8000.0458984375 -> 0.10103759169578552
- link torso_fixed_column_link: mass 16000.0 -> 48.89500045776367
- link torso_fixed_link: mass 16006.1806640625 -> 16.431100845336914
